File: eMonTx.kicad_pcb (KiCad board)
At the start: 2 copper layers, 100 x 100 mm, 38 parts, among them J1 RJ45_LEDS

Commit message: Updated
Parts:
- added Q1: BSS138, TO_SOT_Packages_SMD:SOT-23_Handsoldering, F.Cu at (156.5, 112.2)
- added Q2: BSS138, TO_SOT_Packages_SMD:SOT-23_Handsoldering, F.Cu at (150.7, 112.2)
- added R11: 10K, Resistors_SMD:R_1206_HandSoldering, F.Cu at (151.3, 102.8)
- added R12: 10K, Resistors_SMD:R_1206_HandSoldering, F.Cu at (144.4, 106.0)
- added R13: 10K, Resistors_SMD:R_1206_HandSoldering, F.Cu at (144.3, 102.8)
- added R14: 10K, Resistors_SMD:R_1206_HandSoldering, F.Cu at (134.9, 112.2)
- added R18: 10K, Resistors_SMD:R_1206_HandSoldering, F.Cu at (137.1, 106.0)
- added R7: 10K, Resistors_SMD:R_1206_HandSoldering, F.Cu at (160.8, 112.0)
- added R8: 10K, Resistors_SMD:R_1206_HandSoldering, F.Cu at (158.7, 106.0)
- added R9: 10K, Resistors_SMD:R_1206_HandSoldering, F.Cu at (151.2, 106.2)
- added Rpull1: 4.7K, Resistors_SMD:R_1206_HandSoldering, F.Cu at (136.9, 102.6)
- added Rpull2: 4.7K, Resistors_SMD:R_1206_HandSoldering, F.Cu at (158.3, 102.8)
- moved G*** 15.7 mm to (175.4, 122.6)
- moved G*** 13.6 mm to (121.6, 123.1)
- moved J1 10.3 mm to (146.6, 136.7)
- moved LED1 10.3 mm to (142.3, 117.9)
- moved R10 10.3 mm to (153.5, 117.9)
Connections:
- net /AREF renamed Net-(A1-Pad18)
- net /DIG10 renamed Net-(A1-Pad13)
- net /DIG2 renamed Net-(A1-Pad5)
- net /DIG3 renamed Net-(A1-Pad6)
- net /DIG4 renamed Net-(A1-Pad7)
- net /DIG5 renamed Net-(A1-Pad8)
- net /DIG6 renamed Net-(A1-Pad9)
- net /DIG7 renamed Net-(A1-Pad10)
- net /MISO renamed Net-(A1-Pad15)
- net /MOSI renamed Net-(A1-Pad14)
- net /RESET renamed Net-(A1-Pad3)
- net /RX renamed Net-(A1-Pad1)
- net /SCK renamed Net-(A1-Pad16)
- net /TX renamed Net-(A1-Pad2)
- net /VIN renamed Net-(A1-Pad30)
- A1 pad 17: +3.3VADC -> Net-(A1-Pad17)
- A1 pad 23: /SDA -> /SCL-HV
- A1 pad 24: /SCL -> /SDA-HV
- CT1 pad 4: Net-(CT1-Pad4) -> GND
- CT2 pad 4: Net-(CT2-Pad4) -> GND
- CT3 pad 4: Net-(CT3-Pad4) -> GND
- CT4 pad 4: Net-(CT4-Pad4) -> GND
- J1 pad 1: /SDA -> /SDA-LV
- J1 pad 2: /SCL -> /SCL-LV
Routing:
- net GND: track 246.6 -> 97.2 mm, vias 5 -> 3
- net /SCL: track 82.3 -> 0.00 mm, vias 2 -> 0
- net /SDA: track 73.2 -> 0.00 mm, vias 2 -> 0
- net /SDA-HV: track 0.00 -> 66.3 mm, vias 0 -> 2
- net /SCL-HV: track 0.00 -> 53.3 mm, vias 0 -> 5
- net +3.3VADC: track 74.9 -> 127.4 mm, vias 2 -> 5
- net /ADC3: track 94.2 -> 46.0 mm, vias 0 -> 4
- net /SCL-LV: track 0.00 -> 35.2 mm
- net +5V: track 200.9 -> 230.1 mm, vias 4 -> 8
- net /SDA-LV: track 0.00 -> 27.7 mm, vias 0 -> 2
- net /ADC2: track 60.0 -> 38.2 mm, vias 0 -> 1
- net /LV3: track 0.00 -> 12.1 mm, vias 0 -> 1
- net Net-(C3-Pad1): track 114.2 -> 102.4 mm
- net /LV4: track 0.00 -> 11.5 mm, vias 0 -> 2
- net /HV3: track 0.00 -> 9.23 mm, vias 0 -> 2
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Other:
- board size 100 x 100 mm -> 100 x 90 mm
- board text added: "Cognisense Current Sensor Rev001"
- board text removed: "Cognisense"
