File: eMonTx.sch (KiCad schematic (older format))
At the start: 28 parts, among them J1 RJ45_LEDS

Commit message: Updated
Parts:
- added Q1, Q2: BSS138, TO_SOT_Packages_SMD:SOT-23_Handsoldering, symbol BSS138
- added R11, R7, R8, R9: 10K, Resistors_SMD:R_1206_HandSoldering, symbol R
- added Rpull1, Rpull2: 4.7K, Resistors_SMD:R_1206_HandSoldering, symbol R
Connections:
- net labels added: SCL-HV, SCL-LV, SDA-HV, SDA-LV
- net labels removed: AREF, DIG10, DIG2, DIG3, DIG4, DIG5, DIG6, DIG7, MISO, MOSI, RESET, RX, SCK, SCL, SDA, TX, VIN
- wire segments 94 -> 100
Other:
- note added: "16/4/2018"
- note added: "Cognisense Current Sensor Schematics"
- moved on the sheet: A1
